Commit message: Renamed main xacro file

File: mobile_robot/urdf/mobile_bot.urdf.xacro (robot description, xacro)
@@ -2,11 +2,23 @@
 <robot xmlns:xacro="http://www.ros.org/wiki/xacro" name="mobile_bot">
     <!-- Xacro properties -->
-    <xacro:property name="body_len" value="0.4"/>
-    <xacro:property name="body_width" value="0.2"/>
-    <xacro:property name="body_height" value="0.2"/>
-    <xacro:property name="wheel_diam" value="0.2"/>
+    <xacro:property name="body_len" value="0.325"/>
+    <xacro:property name="body_width" value="0.340"/>
+    <xacro:property name="body_height" value="0.1345"/>
+    <xacro:property name="clearance" value="0.025"/>
+    <xacro:property name="half_body_len" value="${body_len/2.0}"/>
+    <xacro:property name="half_body_height" value="${body_height/2.0}"/>
+    <xacro:property name="bodyOz" value="${half_body_height + clearance}"/>
+    <xacro:property name="wheel_diam" value="0.1016"/>
     <xacro:property name="wheel_rad" value="${wheel_diam/2.0}"/>
-    <xacro:property name="wheel_width" value="0.05"/>
+    <xacro:property name="wheel_width" value="0.025"/>
     <xacro:property name="wheel_sep" value="${body_width - wheel_width}"/>
+    <xacro:property name="wheelOx" value="${wheel_rad - half_body_len}"/>
+    <xacro:property name="wheelOy" value="${wheel_sep/2.0}"/>
+    <xacro:property name="wheelOz" value="${wheel_rad - bodyOz}"/>
+    <xacro:property name="castor_diam" value="0.050"/>
+    <xacro:property name="castor_rad" value="${castor_diam/2.0}"/>
+    <xacro:property name="wheel_to_castor" value="0.2415"/>
+    <xacro:property name="castorOx" value="${wheel_to_castor + wheelOx}"/>
+    <xacro:property name="castorOz" value="${castor_rad - bodyOz}"/>
     <xacro:property name="pi" value="3.14159265359"/>
     <material name="blue">
@@ -28,5 +40,7 @@
     </xacro:macro>
     <!-- Robot base link -->
-    <link name="base_link">
+    <link name="base_link"/>
+    <!-- Robot Body Link -->
+    <link name="body_link">
         <visual>
             <geometry>
@@ -42,7 +56,11 @@
         <xacro:default_inertial mass="20"/>
     </link>
+    <joint name="body_joint" type="fixed">
+        <parent link="base_link"/>
+        <child link="body_link"/>
+    </joint>
     <!-- Wheel macro -->
     <xacro:macro name="wheel" params="prefix reflect">
-        <link name="${prefix}_wheel">
+        <link name="${prefix}_wheel_link">
             <visual>
                 <geometry>
@@ -60,11 +78,11 @@
         <joint name="${prefix}_wheel_joint" type="continuous">
             <axis xyz="0 0 1"/>
-            <parent link="base_link"/>
-            <child link="${prefix}_wheel"/>
-            <origin xyz="${body_len/2.0 - body_len/3.0} ${reflect*wheel_sep/2.0} ${-wheel_rad}" rpy="${pi/2.0} 0 0"/>
+            <parent link="body_link"/>
+            <child link="${prefix}_wheel_link"/>
+            <origin xyz="${wheelOx} ${reflect*wheelOy} ${wheelOz}" rpy="${pi/2.0} 0 0"/>
             <limit effort="100" velocity="15"/>
             <joint_properties damping="0.0" friction="0.0"/>
         </joint>
-        <gazebo reference="{prefix}_wheel">
+        <gazebo reference="{prefix}_wheel_link">
             <mu1 value="200.0"/>
             <mu2 value="100.0"/>
@@ -86,8 +104,8 @@
     <xacro:wheel prefix="right" reflect="-1"/>
     <!-- Front castor -->
-    <link name="castor">
+    <link name="castor_link">
         <visual>
             <geometry>
-                <sphere radius="${wheel_rad/2.0}"/>
+                <sphere radius="${castor_rad}"/>
             </geometry>
             <material name="black"/>
@@ -95,5 +113,5 @@
         <collision>
             <geometry>
-                <sphere radius="${wheel_rad/2.0}"/>
+                <sphere radius="${castor_rad}"/>
             </geometry>
         </collision>
@@ -101,12 +119,14 @@
     </link>
     <joint name="castor_joint" type="fixed">
-        <parent link="base_link"/>
-        <child link="castor"/>
-        <origin xyz="${wheel_rad/2.0 - body_len/2.0} 0 ${-1.5*wheel_rad}" rpy="0 0 0"/>
+        <parent link="body_link"/>
+        <child link="castor_link"/>
+        <origin xyz="${castorOx} 0 ${castorOz}" rpy="0 0 0"/>
     </joint>
-    <gazebo reference="castor">
+    <gazebo reference="castor_link">
         <mu1 value="0.0"/>
         <mu2 value="0.0"/>
     </gazebo>
+    <xacro:include filename="$(find mobile_robot)/urdf/mobile_bot_camera.urdf.xacro" />
+    <xacro:include filename="$(find mobile_robot)/urdf/mobile_bot_laser.urdf.xacro" />
     <!-- Gazebo plugin for ROS Control -->
     <gazebo>

Commit message: Added comments

File: mobile_robot/urdf/mobile_bot.urdf.xacro (robot description, xacro)
@@ -2,4 +2,5 @@
 <robot xmlns:xacro="http://www.ros.org/wiki/xacro" name="mobile_bot">
     <!-- Xacro properties -->
+    <!-- Body dimensions -->
     <xacro:property name="body_len" value="0.325"/>
     <xacro:property name="body_width" value="0.340"/>
@@ -9,4 +10,5 @@
     <xacro:property name="half_body_height" value="${body_height/2.0}"/>
     <xacro:property name="bodyOz" value="${half_body_height + clearance}"/>
+    <!-- Wheel dimensions -->
     <xacro:property name="wheel_diam" value="0.1016"/>
     <xacro:property name="wheel_rad" value="${wheel_diam/2.0}"/>
@@ -16,4 +18,5 @@
     <xacro:property name="wheelOy" value="${wheel_sep/2.0}"/>
     <xacro:property name="wheelOz" value="${wheel_rad - bodyOz}"/>
+    <!-- Castor dimensions -->
     <xacro:property name="castor_diam" value="0.050"/>
     <xacro:property name="castor_rad" value="${castor_diam/2.0}"/>
@@ -21,5 +24,6 @@
     <xacro:property name="castorOx" value="${wheel_to_castor + wheelOx}"/>
     <xacro:property name="castorOz" value="${castor_rad - bodyOz}"/>
-    <xacro:property name="pi" value="3.14159265359"/>
+    <xacro:property name="M_PI" value="3.14159265359"/>
+    <!-- Material Definitions -->
     <material name="blue">
         <color rgba="0 0 0.8 1"/>
@@ -31,4 +35,5 @@
         <color rgba="1 1 1 1"/>
     </material>
+    <!-- Default Inertial macro -->
     <xacro:macro name="default_inertial" params="mass">
         <inertial>
@@ -80,5 +85,5 @@
             <parent link="body_link"/>
             <child link="${prefix}_wheel_link"/>
-            <origin xyz="${wheelOx} ${reflect*wheelOy} ${wheelOz}" rpy="${pi/2.0} 0 0"/>
+            <origin xyz="${wheelOx} ${reflect*wheelOy} ${wheelOz}" rpy="${M_PI/2.0} 0 0"/>
             <limit effort="100" velocity="15"/>
             <joint_properties damping="0.0" friction="0.0"/>
@@ -101,4 +106,5 @@
         </transmission>
     </xacro:macro>
+    <!-- Wheels -->
     <xacro:wheel prefix="left" reflect="1"/>
     <xacro:wheel prefix="right" reflect="-1"/>
@@ -123,8 +129,10 @@
         <origin xyz="${castorOx} 0 ${castorOz}" rpy="0 0 0"/>
     </joint>
+    <!-- Tell Gazebo it has 0 friction -->
     <gazebo reference="castor_link">
         <mu1 value="0.0"/>
         <mu2 value="0.0"/>
     </gazebo>
+    <!-- Camera and Laser -->
     <xacro:include filename="$(find mobile_robot)/urdf/mobile_bot_camera.urdf.xacro" />
     <xacro:include filename="$(find mobile_robot)/urdf/mobile_bot_laser.urdf.xacro" />

Commit message: Adjusted joint frames to face positive x direction

File: mobile_robot/urdf/mobile_bot.urdf.xacro (robot description, xacro)
@@ -15,5 +15,5 @@
     <xacro:property name="wheel_width" value="0.025"/>
     <xacro:property name="wheel_sep" value="${body_width - wheel_width}"/>
-    <xacro:property name="wheelOx" value="${wheel_rad - half_body_len}"/>
+    <xacro:property name="wheelOx" value="${half_body_len - wheel_rad}"/>
     <xacro:property name="wheelOy" value="${wheel_sep/2.0}"/>
     <xacro:property name="wheelOz" value="${wheel_rad - bodyOz}"/>
@@ -22,5 +22,5 @@
     <xacro:property name="castor_rad" value="${castor_diam/2.0}"/>
     <xacro:property name="wheel_to_castor" value="0.2415"/>
-    <xacro:property name="castorOx" value="${wheel_to_castor + wheelOx}"/>
+    <xacro:property name="castorOx" value="${wheelOx - wheel_to_castor}"/>
     <xacro:property name="castorOz" value="${castor_rad - bodyOz}"/>
     <xacro:property name="M_PI" value="3.14159265359"/>
@@ -85,5 +85,5 @@
             <parent link="body_link"/>
             <child link="${prefix}_wheel_link"/>
-            <origin xyz="${wheelOx} ${reflect*wheelOy} ${wheelOz}" rpy="${M_PI/2.0} 0 0"/>
+            <origin xyz="${wheelOx} ${reflect*wheelOy} ${wheelOz}" rpy="${-M_PI/2.0} 0 0"/>
             <limit effort="100" velocity="15"/>
             <joint_properties damping="0.0" friction="0.0"/>

File: mobile_robot/urdf/mobile_bot_camera.urdf.xacro (robot description, xacro)
@@ -4,5 +4,5 @@
     <xacro:include filename="$(find realsense2_description)/urdf/_d435.urdf.xacro"/>
     <xacro:sensor_d435 parent="body_link" use_nominal_extrinsics="true">
-        <origin xyz="${-half_body_len} 0 ${half_body_height}" rpy="0 0 ${M_PI}"/>
+        <origin xyz="${half_body_len} 0 ${half_body_height}" rpy="0 0 0"/>
     </xacro:sensor_d435>
     <xacro:property name="link_name" value="camera_link" />

File: mobile_robot/urdf/mobile_bot_laser.urdf.xacro (robot description, xacro)
@@ -28,5 +28,5 @@
         <parent link="body_link" />
         <child link="laser_mount_link" />
-        <origin xyz="0 0 ${laser_mountOz}" rpy="0 0 0" />
+        <origin xyz="0 0 ${laser_mountOz}" rpy="0 0 ${M_PI}" />
     </joint>
     <!-- Laser link -->
