Commit message: Changed camera name

File: mobile_bot/urdf/mobile_bot/mobile_bot_camera.urdf.xacro (robot description, xacro)
@@ -7,5 +7,5 @@
     </xacro:sensor_d435>
     <xacro:property name="link_name" value="camera_link" />
-    <xacro:property name="camera_name" value="realsense2_d435" />
+    <xacro:property name="camera_name" value="camera" />
     <!-- Gazebo Sensor Plugin for Depth Camera -->
     <gazebo reference="${link_name}">
